Commit message: add camera to my_robot

File: catkin_ws/src/my_robot/urdf/my_robot.xacro (robot description, xacro)
@@ -7,4 +7,28 @@
     <child link="chassis" />
   </joint>
+  <link name='camera'>
+    <pose>0 0 0 0 0 0</pose>
+    <inertial>
+      <mass value=".1"/>
+      <origin xyz=".05 0.05 0.05" rpy=" 0 0 0"/>
+      <inertia
+              ixx="1e-6" ixy="0" ixz="0"
+              iyy="1e-6" iyz="0"
+              izz="1e-6"
+      />
+    </inertial>
+    <collision name='collision'>
+      <origin xyz="0 0 0" rpy=" 0 0 0"/>
+      <geometry>
+        <box size=".05 .05 .05"/>
+      </geometry>
+    </collision>
+    <visual name='visual'>
+      <origin xyz="0 0 0" rpy=" 0 0 0"/>
+      <geometry>
+        <box size=".05 .05 .05"/>
+      </geometry>
+    </visual>
+  </link>
   <link name='left_wheel'>
     <pose>0 0 0 0 0 0</pose>
@@ -119,3 +143,9 @@
     <dynamics damping="1.0" friction="1.0"/>
   </joint>
+  <joint type="fixed" name="camera_joint">
+    <origin xyz=".2 0 0" rpy="0 0 0"/>
+    <child link="camera"/>
+    <parent link="chassis"/>
+    <axis xyz="0 1 0" rpy="0 0 0"/>
+  </joint>
 </robot>

Commit message: add hoyuko lidar to my_robot and use a mesh for the visual geometry

File: catkin_ws/src/my_robot/urdf/my_robot.xacro (robot description, xacro)
@@ -28,4 +28,28 @@
       <geometry>
         <box size=".05 .05 .05"/>
+      </geometry>
+    </visual>
+  </link>
+  <link name='hokuyo'>
+    <pose>0 0 0 0 0 0</pose>
+    <inertial>
+      <mass value="1e-5"/>
+      <origin xyz=".0 .0 .0" rpy=" 0 0 0"/>
+      <inertia
+              ixx="1e-6" ixy="0" ixz="0"
+              iyy="1e-6" iyz="0"
+              izz="1e-6"
+      />
+    </inertial>
+    <collision name='collision'>
+      <origin xyz="0 0 0" rpy=" 0 0 0"/>
+      <geometry>
+        <box size=".1 .1 .1"/>
+      </geometry>
+    </collision>
+    <visual name='visual'>
+      <origin xyz="0 0 0" rpy=" 0 0 0"/>
+      <geometry>
+        <mesh filename="package://my_robot/meshes/hokuyo.dae"/>
       </geometry>
     </visual>
@@ -149,3 +173,9 @@
     <axis xyz="0 1 0" rpy="0 0 0"/>
   </joint>
+  <joint type="fixed" name="hokuyo_joint">
+    <origin xyz=".15 0 .1" rpy="0 0 0"/>
+    <child link="hokuyo"/>
+    <parent link="chassis"/>
+    <axis xyz="0 1 0" rpy="0 0 0"/>
+  </joint>
 </robot>

Commit message: add color blue to chassis for gazebo visualization

File: catkin_ws/src/my_robot/urdf/my_robot.xacro (robot description, xacro)
@@ -7,4 +7,7 @@
     <child link="chassis" />
   </joint>
+  <gazebo reference="chassis">
+    <material>Gazebo/Blue</material>
+  </gazebo>
   <link name='camera'>
     <pose>0 0 0 0 0 0</pose>

Commit message: modify my_robot size and remove one caster wheel

File: catkin_ws/src/my_robot/urdf/my_robot.xacro (robot description, xacro)
@@ -9,4 +9,10 @@
   </joint>
   <gazebo reference="chassis">
+    <material>Gazebo/Green</material>
+  </gazebo>
+  <gazebo reference="left_wheel">
+    <material>Gazebo/Blue</material>
+  </gazebo>
+  <gazebo reference="right_wheel">
     <material>Gazebo/Blue</material>
   </gazebo>
@@ -25,5 +31,5 @@
       <origin xyz="0 0 0" rpy=" 0 0 0"/>
       <geometry>
-        <box size=".05 .05 .05"/>
+        <box size=".025 .025 .025"/>
       </geometry>
     </collision>
@@ -31,5 +37,5 @@
       <origin xyz="0 0 0" rpy=" 0 0 0"/>
       <geometry>
-        <box size=".05 .05 .05"/>
+        <box size=".025 .025 .025"/>
       </geometry>
     </visual>
@@ -49,5 +55,5 @@
       <origin xyz="0 0 0" rpy=" 0 0 0"/>
       <geometry>
-        <box size=".1 .1 .1"/>
+        <box size=".05 .05 .05"/>
       </geometry>
     </collision>
@@ -62,5 +68,5 @@
     <pose>0 0 0 0 0 0</pose>
     <inertial>
-      <mass value="5.0"/>
+      <mass value="2.0"/>
       <origin xyz="0.0 0 0" rpy=" 0 0 0"/>
       <inertia
@@ -73,5 +79,5 @@
       <origin xyz="0 0 0" rpy=" 0 1.5707 1.5707"/>
       <geometry>
-        <cylinder radius=".1" length=".05"/>
+        <cylinder radius=".05" length=".03"/>
       </geometry>
     </collision>
@@ -79,5 +85,5 @@
       <origin xyz="0 0 0" rpy=" 0 1.5707 1.5707"/>
       <geometry>
-        <cylinder radius=".1" length=".05"/>
+        <cylinder radius=".05" length=".03"/>
       </geometry>
     </visual>
@@ -86,5 +92,5 @@
     <pose>0 0 0 0 0 0</pose>
     <inertial>
-      <mass value="5.0"/>
+      <mass value="2.0"/>
       <origin xyz="0.0 0 0" rpy=" 0 0 0"/>
       <inertia
@@ -97,5 +103,5 @@
       <origin xyz="0 0 0" rpy=" 0 1.5707 1.5707"/>
       <geometry>
-        <cylinder radius=".1" length=".05"/>
+        <cylinder radius=".05" length=".03"/>
       </geometry>
     </collision>
@@ -103,5 +109,5 @@
       <origin xyz="0 0 0" rpy=" 0 1.5707 1.5707"/>
       <geometry>
-        <cylinder radius=".1" length=".05"/>
+        <cylinder radius=".05" length=".03"/>
       </geometry>
     </visual>
@@ -121,5 +127,5 @@
       <origin xyz="0 0 0" rpy=" 0 0 0"/>
       <geometry>
-        <box size=".4 .2 .1"/>
+        <box size=".2 .1 .05"/>
       </geometry>
     </collision>
@@ -127,34 +133,22 @@
       <origin xyz="0 0 0" rpy=" 0 0 0"/>
       <geometry>
-        <box size=".4 .2 .1"/>
+        <box size=".2 .1 .05"/>
       </geometry>
     </visual>
     <collision name='back_caster_collision'>
-      <origin xyz="-0.15 0 -0.05" rpy=" 0 0 0"/>
+      <origin xyz="-0.075 0 -0.025" rpy=" 0 0 0"/>
       <geometry>
-        <sphere radius="0.0499"/>
+        <sphere radius="0.02499"/>
       </geometry>
     </collision>
     <visual name='back_caster_visual'>
-      <origin xyz="-0.15 0 -0.05" rpy=" 0 0 0"/>
+      <origin xyz="-0.075 0 -0.025" rpy=" 0 0 0"/>
       <geometry>
-        <sphere radius="0.05"/>
-      </geometry>
-    </visual>
-    <collision name='front_caster_collision'>
-      <origin xyz="0.15 0 -0.05" rpy=" 0 0 0"/>
-      <geometry>
-        <sphere radius="0.0499"/>
-      </geometry>
-    </collision>
-    <visual name='front_caster_visual'>
-      <origin xyz="0.15 0 -0.05" rpy=" 0 0 0"/>
-      <geometry>
-        <sphere radius="0.05"/>
+        <sphere radius="0.025"/>
       </geometry>
     </visual>
   </link>
   <joint type="continuous" name="left_wheel_hinge">
-    <origin xyz="0 0.15 0" rpy="0 0 0"/>
+    <origin xyz="0.03 0.075 0" rpy="0 0 0"/>
     <child link="left_wheel"/>
     <parent link="chassis"/>
@@ -164,5 +158,5 @@
   </joint>
   <joint type="continuous" name="right_wheel_hinge">
-    <origin xyz="0 -0.15 0" rpy="0 0 0"/>
+    <origin xyz="0.03 -0.075 0" rpy="0 0 0"/>
     <child link="right_wheel"/>
     <parent link="chassis"/>
@@ -172,5 +166,5 @@
   </joint>
   <joint type="fixed" name="camera_joint">
-    <origin xyz=".2 0 0" rpy="0 0 0"/>
+    <origin xyz=".1 0 0" rpy="0 0 0"/>
     <child link="camera"/>
     <parent link="chassis"/>
@@ -178,5 +172,5 @@
   </joint>
   <joint type="fixed" name="hokuyo_joint">
-    <origin xyz=".15 0 .1" rpy="0 0 0"/>
+    <origin xyz=".075 0 .05" rpy="0 0 0"/>
     <child link="hokuyo"/>
     <parent link="chassis"/>

Commit message: reduce velocity to allow better following of ball

File: catkin_ws/src/my_robot/urdf/my_robot.xacro (robot description, xacro)
@@ -150,5 +150,5 @@
   </link>
   <joint type="continuous" name="left_wheel_hinge">
-    <origin xyz="0.03 0.075 0" rpy="0 0 0"/>
+    <origin xyz="0.04 0.075 0" rpy="0 0 0"/>
     <child link="left_wheel"/>
     <parent link="chassis"/>
@@ -158,5 +158,5 @@
   </joint>
   <joint type="continuous" name="right_wheel_hinge">
-    <origin xyz="0.03 -0.075 0" rpy="0 0 0"/>
+    <origin xyz="0.04 -0.075 0" rpy="0 0 0"/>
     <child link="right_wheel"/>
     <parent link="chassis"/>
