Commit message: add camera optical joint and link to robot xacro

File: Project4/catkin_ws/src/my_robot/urdf/my_robot.xacro (robot description, xacro)
@@ -171,4 +171,10 @@
     <axis xyz="0 1 0" rpy="0 0 0"/>
   </joint>
+  <joint name="camera_optical_joint" type="fixed">
+    <origin xyz="0 0 0" rpy="-1.5707 0 -1.5707"/>
+    <parent link="camera"/>
+    <child link="camera_link_optical"/>
+  </joint>
+  <link name="camera_link_optical"/>
   <joint type="fixed" name="hokuyo_joint">
     <origin xyz=".075 0 .05" rpy="0 0 0"/>

Commit message: fix 3d camera settings

File: Project4/catkin_ws/src/my_robot/urdf/my_robot.xacro (robot description, xacro)
@@ -173,5 +173,5 @@
   <joint name="camera_optical_joint" type="fixed">
     <origin xyz="0 0 0" rpy="-1.5707 0 -1.5707"/>
-    <parent link="camera"/>
+    <parent link="camera_link"/>
     <child link="camera_link_optical"/>
   </joint>

Commit message: revert changes in 3d camera

File: Project4/catkin_ws/src/my_robot/urdf/my_robot.xacro (robot description, xacro)
@@ -173,5 +173,5 @@
   <joint name="camera_optical_joint" type="fixed">
     <origin xyz="0 0 0" rpy="-1.5707 0 -1.5707"/>
-    <parent link="camera_link"/>
+    <parent link="camera"/>
     <child link="camera_link_optical"/>
   </joint>

Commit message: recover example robot

File: Project4/catkin_ws/src/my_robot/urdf/my_robot.xacro (robot description, xacro)
@@ -31,5 +31,5 @@
       <origin xyz="0 0 0" rpy=" 0 0 0"/>
       <geometry>
-        <box size=".025 .025 .025"/>
+        <box size=".05 .05 .05"/>
       </geometry>
     </collision>
@@ -37,5 +37,5 @@
       <origin xyz="0 0 0" rpy=" 0 0 0"/>
       <geometry>
-        <box size=".025 .025 .025"/>
+        <box size=".05 .05 .05"/>
       </geometry>
     </visual>
@@ -55,5 +55,5 @@
       <origin xyz="0 0 0" rpy=" 0 0 0"/>
       <geometry>
-        <box size=".05 .05 .05"/>
+        <box size=".1 .1 .1"/>
       </geometry>
     </collision>
@@ -127,5 +127,5 @@
       <origin xyz="0 0 0" rpy=" 0 0 0"/>
       <geometry>
-        <box size=".2 .1 .05"/>
+        <box size=".4 .2 .1"/>
       </geometry>
     </collision>
@@ -133,22 +133,34 @@
       <origin xyz="0 0 0" rpy=" 0 0 0"/>
       <geometry>
-        <box size=".2 .1 .05"/>
+        <box size=".4 .2 .1"/>
       </geometry>
     </visual>
     <collision name='back_caster_collision'>
-      <origin xyz="-0.075 0 -0.025" rpy=" 0 0 0"/>
+      <origin xyz="-0.15 0 -0.05" rpy=" 0 0 0"/>
       <geometry>
-        <sphere radius="0.02499"/>
+        <sphere radius="0.0499"/>
       </geometry>
     </collision>
     <visual name='back_caster_visual'>
-      <origin xyz="-0.075 0 -0.025" rpy=" 0 0 0"/>
+      <origin xyz="-0.15 0 -0.05" rpy=" 0 0 0"/>
       <geometry>
-        <sphere radius="0.025"/>
+        <sphere radius="0.05"/>
+      </geometry>
+    </visual>
+    <collision name='front_caster_collision'>
+      <origin xyz="0.15 0 -0.05" rpy=" 0 0 0"/>
+      <geometry>
+        <sphere radius="0.0499"/>
+      </geometry>
+    </collision>
+    <visual name='front_caster_visual'>
+      <origin xyz="0.15 0 -0.05" rpy=" 0 0 0"/>
+      <geometry>
+        <sphere radius="0.05"/>
       </geometry>
     </visual>
   </link>
   <joint type="continuous" name="left_wheel_hinge">
-    <origin xyz="0.04 0.075 0" rpy="0 0 0"/>
+    <origin xyz="0 0.15 0" rpy="0 0 0"/>
     <child link="left_wheel"/>
     <parent link="chassis"/>
@@ -158,5 +170,5 @@
   </joint>
   <joint type="continuous" name="right_wheel_hinge">
-    <origin xyz="0.04 -0.075 0" rpy="0 0 0"/>
+    <origin xyz="0 -0.15 0" rpy="0 0 0"/>
     <child link="right_wheel"/>
     <parent link="chassis"/>
@@ -166,5 +178,5 @@
   </joint>
   <joint type="fixed" name="camera_joint">
-    <origin xyz=".1 0 0" rpy="0 0 0"/>
+    <origin xyz=".2 0 0" rpy="0 0 0"/>
     <child link="camera"/>
     <parent link="chassis"/>
@@ -178,5 +190,5 @@
   <link name="camera_link_optical"/>
   <joint type="fixed" name="hokuyo_joint">
-    <origin xyz=".075 0 .05" rpy="0 0 0"/>
+    <origin xyz=".15 0 .1" rpy="0 0 0"/>
     <child link="hokuyo"/>
     <parent link="chassis"/>

Commit message: make robot more stable

File: Project4/catkin_ws/src/my_robot/urdf/my_robot.xacro (robot description, xacro)
@@ -148,7 +148,19 @@
       </geometry>
     </visual>
+    <collision name='front_caster_collision'>
+      <origin xyz="0.075 0 -0.025" rpy=" 0 0 0"/>
+      <geometry>
+        <sphere radius="0.02499"/>
+      </geometry>
+    </collision>
+    <visual name='front_caster_visual'>
+      <origin xyz="0.075 0 -0.025" rpy=" 0 0 0"/>
+      <geometry>
+        <sphere radius="0.025"/>
+      </geometry>
+    </visual>
   </link>
   <joint type="continuous" name="left_wheel_hinge">
-    <origin xyz="0.04 0.075 0" rpy="0 0 0"/>
+    <origin xyz="0.0 0.075 0.0" rpy="0 0 0"/>
     <child link="left_wheel"/>
     <parent link="chassis"/>
@@ -158,5 +170,5 @@
   </joint>
   <joint type="continuous" name="right_wheel_hinge">
-    <origin xyz="0.04 -0.075 0" rpy="0 0 0"/>
+    <origin xyz="0.0 -0.0749 0.0" rpy="0 0 0"/>
     <child link="right_wheel"/>
     <parent link="chassis"/>
